File: ThumbsUp.kicad_pcb (KiCad board)
At the start: 2 copper layers, 250.8 x 270.5 mm, 170 parts, among them IC1 RP2040, IC2 W25Q128JVSIM, IC3 RP2040, IC4 W25Q128JVSIM, J1 Conn_01x04_Male, J10 Raiser_Male, J11 Raiser_Female, J12 Raiser_Male, J13 Raiser_Female, J14 Raiser_Male, J15 Raiser_Female, J16 Raiser_Male, J17 Raiser_Female, J18 Raiser_Male, J19 Raiser_Female, J2 Conn_01x04_Male, J20 Conn_01x04_Female, J21 Conn_01x04_Female, J22 Conn_01x04_Female, J23 Conn_01x04_Female, J24 Conn_01x04_Male, J25 Conn_01x04_Male, J26 Conn_01x04_Male, J27 Conn_01x04_Male, J28 Conn_01x04_Female, J29 Conn_01x04_Female, J3 Conn_01x04_Female, J30 Conn_01x04_Female, J31 Conn_01x04_Female, J32 USB_C_Receptacle_USB2.0, J33 Raiser_Male, J34 Raiser_Female, J35 Raiser_Male, J36 STX-3501-3N, J37 USB_C_Receptacle_USB2.0, J38 Raiser_Female, J39 Raiser_Male, J4 Conn_01x04_Male, J40 Raiser_Female, J41 Raiser_Male, J42 Raiser_Female, J43 Raiser_Male, J44 Raiser_Female, J45 Raiser_Male, J46 STX-3501-3N, J47 Raiser_Female, J48 Raiser_Male, J49 Raiser_Female, J5 Conn_01x04_Female, J50 Raiser_Male, J51 Raiser_Female, J52 Raiser_Male, J6 Conn_01x04_Male, J7 Conn_01x04_Male, J8 Conn_01x04_Male, J9 Raiser_Female, U1 AMS1117-3.3_SOT223, U2 AMS1117-3.3_SOT223, Y1 ABLS-12.000MHZ-B4-T, Y2 ABLS-12.000MHZ-B4-T

Commit message: Removed the top row in schematics and PCBs, redrew the tracks
Parts:
- removed G***: LOGO, Silkscreens:Crowfeet75
- removed J2, J25: Conn_01x04_Male, Connector_PinHeader_2.54mm:PinHeader_1x04_P2.54mm_Vertical
- removed J21, J29: Conn_01x04_Female, Connector_PinSocket_2.54mm:PinSocket_1x04_P2.54mm_Vertical
- removed MX45: SwGrave, MX_Alps_Hybrid:MX-1U-NoLED_HotSwap
- removed MX46: Sw1, MX_Alps_Hybrid:MX-1U-NoLED_HotSwap
- removed MX47: Sw2, MX_Alps_Hybrid:MX-1U-NoLED_HotSwap
- removed MX48: Sw3, MX_Alps_Hybrid:MX-1U-NoLED_HotSwap
- removed MX49: Sw4, MX_Alps_Hybrid:MX-1U-NoLED_HotSwap
- removed MX50: Sw5, MX_Alps_Hybrid:MX-1U-NoLED_HotSwap
- removed MX51: Sw6, MX_Alps_Hybrid:MX-1U-NoLED_HotSwap
- removed MX52: Sw7, MX_Alps_Hybrid:MX-1U-NoLED_HotSwap
- removed MX53: Sw8, MX_Alps_Hybrid:MX-1U-NoLED_HotSwap
- removed MX54: Sw9, MX_Alps_Hybrid:MX-1U-NoLED_HotSwap
- removed MX55: Sw0, MX_Alps_Hybrid:MX-1U-NoLED_HotSwap
- removed MX56: SwDEL, MX_Alps_Hybrid:MX-1U-NoLED_HotSwap
- moved F1 34.5 mm to (111.8, 415.5)
- moved F2 23.7 mm to (172.4, 412.0)
- moved J40 19.0 mm to (153.0, 525.9)
- moved J49 19.0 mm to (102.7, 517.2)
- moved J32 19.0 mm to (112.0, 391.2)
- moved J36 19.0 mm to (125.9, 410.2)
- moved J37 19.0 mm to (172.3, 391.1)
- moved J38 19.0 mm to (126.4, 526.1)
- moved J39 19.0 mm to (128.9, 398.7)
- moved J41 19.0 mm to (155.5, 398.4)
- moved J46 19.0 mm to (157.8, 405.1)
- moved J50 19.0 mm to (105.1, 389.8)
- moved J51 19.0 mm to (176.7, 517.4)
- moved J52 19.0 mm to (179.2, 389.9)
- moved R10 19.0 mm to (179.5, 391.7)
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Connections:
- IC1 pad 27: K_4 -> (no net)
- IC1 pad 28: K_5 -> (no net)
- IC1 pad 30: K_GRAVE -> (no net)
- IC1 pad 31: K_1 -> (no net)
- IC1 pad 34: K_2 -> (no net)
- IC1 pad 35: K_3 -> (no net)
- IC3 pad 12: K_6 -> (no net)
- IC3 pad 13: K_DEL -> (no net)
- IC3 pad 14: K_0 -> (no net)
- IC3 pad 27: K_9 -> (no net)
- IC3 pad 28: K_8 -> (no net)
- IC3 pad 35: K_7 -> (no net)
- J39 pad 1: K_5 -> K_T
Routing:
- net L-BASE: track 1024.2 -> 881.2 mm, vias 31 -> 29
- net K_7: track 133.1 -> 0.00 mm, vias 5 -> 0
- net K_4: track 125.5 -> 0.00 mm, vias 1 -> 0
- net K_5: track 123.7 -> 0.00 mm, vias 1 -> 0
- net Net-(J29-Pad4): track 108.5 -> 0.00 mm
- net K_8: track 106.5 -> 0.00 mm, vias 3 -> 0
- net K_9: track 103.9 -> 0.00 mm, vias 3 -> 0
- net K_2: track 102.5 -> 0.00 mm, vias 1 -> 0
- net K_3: track 102.5 -> 0.00 mm, vias 1 -> 0
- net K_1: track 100.2 -> 0.00 mm, vias 1 -> 0
- net K_GRAVE: track 100.2 -> 0.00 mm, vias 1 -> 0
- net Net-(J21-Pad4): track 99.8 -> 0.00 mm
- net K_6: track 88.7 -> 0.00 mm, vias 2 -> 0
- net Net-(J29-Pad3): track 78.7 -> 0.00 mm
- net K_0: track 72.9 -> 0.00 mm, vias 1 -> 0
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Other:
- outline, holes or cut-outs redrawn
- board text added: "u/AK66666 ThumbsUp! v6 MX 2023-06-14"
- board text removed: "u/AK66666 ThumbsUp! v4 MX 2023-05-15"
