File: ThumbsUp.sch (KiCad schematic (older format))
At the start: 169 parts, among them IC1 RP2040, IC2 W25Q128JVSIM, IC3 RP2040, IC4 W25Q128JVSIM, J1 Conn_01x04_Male, J10 Raiser_Male, J11 Raiser_Female, J12 Raiser_Male, J13 Raiser_Female, J14 Raiser_Male, J15 Raiser_Female, J16 Raiser_Male, J17 Raiser_Female, J18 Raiser_Male, J19 Raiser_Female, J2 Conn_01x04_Male, J20 Conn_01x04_Female, J21 Conn_01x04_Female, J22 Conn_01x04_Female, J23 Conn_01x04_Female, J24 Conn_01x04_Male, J25 Conn_01x04_Male, J26 Conn_01x04_Male, J27 Conn_01x04_Male, J28 Conn_01x04_Female, J29 Conn_01x04_Female, J3 Conn_01x04_Female, J30 Conn_01x04_Female, J31 Conn_01x04_Female, J32 USB_C_Receptacle_USB2.0, J33 Raiser_Male, J34 Raiser_Female, J35 Raiser_Male, J36 STX-3501-3N, J37 USB_C_Receptacle_USB2.0, J38 Raiser_Female, J39 Raiser_Male, J4 Conn_01x04_Male, J40 Raiser_Female, J41 Raiser_Male, J42 Raiser_Female, J43 Raiser_Male, J44 Raiser_Female, J45 Raiser_Male, J46 STX-3501-3N, J47 Raiser_Female, J48 Raiser_Male, J49 Raiser_Female, J5 Conn_01x04_Female, J50 Raiser_Male, J51 Raiser_Female, J52 Raiser_Male, J6 Conn_01x04_Male, J7 Conn_01x04_Male, J8 Conn_01x04_Male, J9 Raiser_Female, U1 AMS1117-3.3_SOT223, U2 AMS1117-3.3_SOT223, Y1 ABLS-12.000MHZ-B4-T, Y2 ABLS-12.000MHZ-B4-T

Commit message: Removed the top row in schematics and PCBs, redrew the tracks
Parts:
- removed J2, J25: Conn_01x04_Male, Connector_PinHeader_2.54mm:PinHeader_1x04_P2.54mm_Vertical, symbol Connector:Conn_01x04_Male
- removed J21, J29: Conn_01x04_Female, Connector_PinSocket_2.54mm:PinSocket_1x04_P2.54mm_Vertical, symbol Connector:Conn_01x04_Female
- removed MX45: SwGrave, MX_Alps_Hybrid:MX-1U-NoLED_HotSwap, symbol ThumbsUp-rescue:MX-NoLED-MX_Alps_Hybrid
- removed MX46: Sw1, MX_Alps_Hybrid:MX-1U-NoLED_HotSwap, symbol ThumbsUp-rescue:MX-NoLED-MX_Alps_Hybrid
- removed MX47: Sw2, MX_Alps_Hybrid:MX-1U-NoLED_HotSwap, symbol ThumbsUp-rescue:MX-NoLED-MX_Alps_Hybrid
- removed MX48: Sw3, MX_Alps_Hybrid:MX-1U-NoLED_HotSwap, symbol ThumbsUp-rescue:MX-NoLED-MX_Alps_Hybrid
- removed MX49: Sw4, MX_Alps_Hybrid:MX-1U-NoLED_HotSwap, symbol ThumbsUp-rescue:MX-NoLED-MX_Alps_Hybrid
- removed MX50: Sw5, MX_Alps_Hybrid:MX-1U-NoLED_HotSwap, symbol ThumbsUp-rescue:MX-NoLED-MX_Alps_Hybrid
- removed MX51: Sw6, MX_Alps_Hybrid:MX-1U-NoLED_HotSwap, symbol ThumbsUp-rescue:MX-NoLED-MX_Alps_Hybrid
- removed MX52: Sw7, MX_Alps_Hybrid:MX-1U-NoLED_HotSwap, symbol ThumbsUp-rescue:MX-NoLED-MX_Alps_Hybrid
- removed MX53: Sw8, MX_Alps_Hybrid:MX-1U-NoLED_HotSwap, symbol ThumbsUp-rescue:MX-NoLED-MX_Alps_Hybrid
- removed MX54: Sw9, MX_Alps_Hybrid:MX-1U-NoLED_HotSwap, symbol ThumbsUp-rescue:MX-NoLED-MX_Alps_Hybrid
- removed MX55: Sw0, MX_Alps_Hybrid:MX-1U-NoLED_HotSwap, symbol ThumbsUp-rescue:MX-NoLED-MX_Alps_Hybrid
- removed MX56: SwDEL, MX_Alps_Hybrid:MX-1U-NoLED_HotSwap, symbol ThumbsUp-rescue:MX-NoLED-MX_Alps_Hybrid
Connections:
- net K_T: now also J39.1 (Pin_1)
- net K_0: no longer names the net of IC3.14 (GPIO11)
- net K_1: no longer names the net of IC1.31 (GPIO20)
- net K_2: no longer names the net of IC1.34 (GPIO22)
- net K_3: no longer names the net of IC1.35 (GPIO23)
- net K_4: no longer names the net of IC1.27 (GPIO16)
- net K_5: no longer names the net of IC1.28 (GPIO17)
- net K_5: no longer J39.1 (Pin_1)
- net K_6: no longer names the net of IC3.12 (GPIO9)
- net K_7: no longer names the net of IC3.35 (GPIO23)
- net K_8: no longer names the net of IC3.28 (GPIO17)
- net K_9: no longer names the net of IC3.27 (GPIO16)
- net K_DEL: no longer names the net of IC3.13 (GPIO10)
- net K_GRAVE: no longer names the net of IC1.30 (GPIO19)
- no-connect marks 86 -> 100

Commit message: Re-wired L2 RP2040 and memory as per manual
Parts:
- IC1, IC3: footprint RP2040:QFN40P700X700X90-57N-D -> RP2040_minimal:RP2040-QFN-56
Changed lines of the file:
@@
 F 0 "IC1" H 4294 6546 50  0000 L CNN
 F 1 "RP2040" H 3100 6450 50  0000 L CNN
-F 2 "RP2040:QFN40P700X700X90-57N-D" H 4100 7800 50  0001 L CNN
+F 2 "RP2040_minimal:RP2040-QFN-56" H 4100 7800 50  0001 L CNN
 F 3 "https://datasheets.raspberrypi.org/rp2040/rp2040-datasheet.pdf" H 4100 7700 50  0001 L CNN
 F 4 "Microcontroller in QFN Package" H 4100 7600 50  0001 L CNN "Description"
@@
 F 0 "IC3" H 14594 6496 50  0000 L CNN
 F 1 "RP2040" H 13400 6400 50  0000 L CNN
-F 2 "RP2040:QFN40P700X700X90-57N-D" H 14400 7750 50  0001 L CNN
+F 2 "RP2040_minimal:RP2040-QFN-56" H 14400 7750 50  0001 L CNN
 F 3 "https://datasheets.raspberrypi.org/rp2040/rp2040-datasheet.pdf" H 14400 7650 50  0001 L CNN
 F 4 "Microcontroller in QFN Package" H 14400 7550 50  0001 L CNN "Description"
